Commit message: simplified robot to box with 4 wheels

File: src/rviz_demo/urdf/robot.urdf.xacro (robot description, xacro)
@@ -1,9 +1,7 @@
 <?xml version="1.0"?>
 <robot name="roscontrol" xmlns:xacro="http://ros.org/wiki/xacro">
-  <xacro:property name="width" value="0.2" />
-  <xacro:property name="leglen" value="0.6" />
-  <xacro:property name="polelen" value="0.2" />
-  <xacro:property name="bodylen" value="0.6" />
-  <xacro:property name="baselen" value="0.4" />
+  <xacro:property name="robot_side" value="0.3" />
+  <xacro:property name="lidar_radius" value="0.06" />
+  <xacro:property name="lidar_height" value="0.12" />
   <xacro:property name="wheeldiam" value="0.07" />
   <xacro:property name="pi" value="3.1415" />
@@ -26,5 +24,5 @@
     <visual>
       <geometry>
-        <cylinder radius="${width}" length="${bodylen}"/>
+        <box size="${robot_side} ${robot_side} ${robot_side/2}"/>
       </geometry>
       <material name="blue"/>
@@ -32,15 +30,15 @@
     <collision>
       <geometry>
-        <cylinder radius="${width}" length="${bodylen}"/>
+        <box size="${robot_side} ${robot_side} ${robot_side/2}"/>
       </geometry>
     </collision>
-    <xacro:default_inertial mass="10"/>
+    <xacro:default_inertial mass="30"/>
   </link>
-  <xacro:macro name="wheel" params="prefix suffix reflect">
-    <link name="${prefix}_${suffix}_wheel">
+  <xacro:macro name="wheel" params="rl fb rl_reflect fb_reflect">
+    <link name="${rl}_${fb}_wheel">
       <visual>
         <origin xyz="0 0 0" rpy="${pi/2} 0 0" />
         <geometry>
-          <cylinder radius="${wheeldiam/2}" length="0.1"/>
+          <cylinder radius="${wheeldiam/2}" length="${wheeldiam/4}"/>
         </geometry>
         <material name="black"/>
@@ -49,18 +47,16 @@
         <origin xyz="0 0 0" rpy="${pi/2} 0 0" />
         <geometry>
-          <cylinder radius="${wheeldiam/2}" length="0.1"/>
+          <cylinder radius="${wheeldiam/2}" length="${wheeldiam/4}"/>
         </geometry>
       </collision>
       <xacro:default_inertial mass="1"/>
     </link>
-    <joint name="${prefix}_${suffix}_wheel_joint" type="continuous">
+    <joint name="${rl}_${fb}_wheel_joint" type="continuous">
       <axis xyz="0 1 0" rpy="0 0 0" />
-      <parent link="${prefix}_base"/>
-      <child link="${prefix}_${suffix}_wheel"/>
-      <origin xyz="${baselen*reflect/3} 0 -${wheeldiam/2+.05}" rpy="0 0 0"/>
+      <parent link="base_link"/>
+      <child link="${rl}_${fb}_wheel"/>
+      <origin xyz="${robot_side/3*fb_reflect} ${robot_side/3*rl_reflect} -${wheeldiam/2+.05}" rpy="0 0 0"/>
     </joint>
-    <!-- This block provides the simulator (Gazebo) with information on a few additional
-    physical properties. See http://gazebosim.org/tutorials/?tut=ros_urdf for more-->
-    <gazebo reference="${prefix}_${suffix}_wheel">
+    <gazebo reference="${rl}_${fb}_wheel">
       <mu1 value="200.0"/>
       <mu2 value="100.0"/>
@@ -69,111 +65,34 @@
       <material>Gazebo/Grey</material>
     </gazebo>
-    <!-- This block connects the wheel joint to an actuator (motor), which informs both
-    simulation and visualization of the robot -->
-    <transmission name="${prefix}_${suffix}_wheel_trans">
+    <transmission name="${rl}_${fb}_wheel_trans">
       <type>transmission_interface/SimpleTransmission</type>
-      <actuator name="${prefix}_${suffix}_wheel_motor">
+      <actuator name="${rl}_${fb}_wheel_motor">
         <mechanicalReduction>1</mechanicalReduction>
       </actuator>
-      <joint name="${prefix}_${suffix}_wheel_joint">
+      <joint name="${rl}_${fb}_wheel_joint">
         <hardwareInterface>VelocityJointInterface</hardwareInterface>
       </joint>
     </transmission>
   </xacro:macro>
-  <xacro:macro name="leg" params="prefix reflect">
-    <link name="${prefix}_leg">
-      <visual>
-        <geometry>
-          <box size="${leglen} 0.1 0.2"/>
-        </geometry>
-        <origin xyz="0 0 -${leglen/2}" rpy="0 ${pi/2} 0"/>
-        <material name="white"/>
-      </visual>
-      <collision>
-        <geometry>
-          <box size="${leglen} 0.1 0.2"/>
-        </geometry>
-        <origin xyz="0 0 -${leglen/2}" rpy="0 ${pi/2} 0"/>
-      </collision>
-      <xacro:default_inertial mass="10"/>
-    </link>
-    <joint name="base_to_${prefix}_leg" type="fixed">
-      <parent link="base_link"/>
-      <child link="${prefix}_leg"/>
-      <origin xyz="0 ${reflect*(width+.02)} 0.25" />
-    </joint>
-    <link name="${prefix}_base">
-      <visual>
-        <geometry>
-          <box size="${baselen} 0.1 0.1"/>
-        </geometry>
-        <material name="white"/>
-      </visual>
-      <collision>
-        <geometry>
-          <box size="${baselen} 0.1 0.1"/>
-        </geometry>
-      </collision>
-      <xacro:default_inertial mass="10"/>
-    </link>
-    <joint name="${prefix}_base_joint" type="fixed">
-      <parent link="${prefix}_leg"/>
-      <child link="${prefix}_base"/>
-      <origin xyz="0 0 ${-leglen}" />
-    </joint>
-    <xacro:wheel prefix="${prefix}" suffix="front" reflect="1"/>
-    <xacro:wheel prefix="${prefix}" suffix="back" reflect="-1"/>
-  </xacro:macro>
-  <xacro:leg prefix="right" reflect="-1" />
-  <xacro:leg prefix="left" reflect="1" />
-  <link name="head">
+	<xacro:wheel rl="right" fb="front" rl_reflect="1" fb_reflect="1"/>
+	<xacro:wheel rl="right" fb="back" rl_reflect="1" fb_reflect="-1"/>
+	<xacro:wheel rl="left" fb="front" rl_reflect="-1" fb_reflect="1"/>
+	<xacro:wheel rl="left" fb="back" rl_reflect="-1" fb_reflect="-1"/>
+  <link name="lidar">
     <visual>
       <geometry>
-        <sphere radius="${width}"/>
+        <cylinder radius="${lidar_radius}" length="${lidar_height}" />
       </geometry>
-      <material name="white"/>
+      <material name="blue"/>
+      <origin xyz="0 0 0"/>
     </visual>
     <collision>
       <geometry>
-        <sphere radius="${width}"/>
-      </geometry>
-    </collision>
-    <xacro:default_inertial mass="2"/>
-  </link>
-  <joint name="head_swivel" type="continuous">
-    <parent link="base_link"/>
-    <child link="head"/>
-    <axis xyz="0 0 1"/>
-    <origin xyz="0 0 ${bodylen/2}"/>
-    <limit effort="30" velocity="1.0"/>
-    <dynamics damping="0.0" friction="0.0"/>
-  </joint>
-  <!-- This block connects the head_swivel joint to an actuator (motor), which informs both
-  simulation and visualization of the robot -->
-  <transmission name="head_swivel_trans">
-    <type>transmission_interface/SimpleTransmission</type>
-    <actuator name="$head_swivel_motor">
-      <mechanicalReduction>1</mechanicalReduction>
-    </actuator>
-    <joint name="head_swivel">
-      <hardwareInterface>PositionJointInterface</hardwareInterface>
-    </joint>
-  </transmission>
-  <link name="laser_frame">
-    <visual>
-      <geometry>
-        <box size="0.08 0.08 0.08"/>
-      </geometry>
-      <material name="blue"/>
-      <origin xyz="-0.04 0 0"/>
-    </visual>
-    <collision>
-      <geometry>
-        <box size="0.08 0.08 0.08"/>
+        <cylinder radius="${lidar_radius}" length="${lidar_height}" />
       </geometry>
     </collision>
     <xacro:default_inertial mass="1"/>
   </link>
-	<gazebo reference="laser_frame">
+	<gazebo reference="lidar">
 		<sensor name="laser" type="ray">
 			<pose>0 0 0 0 0 0</pose>
@@ -197,14 +116,13 @@
 			<plugin name="laser_controller" filename="libgazebo_ros_laser.so">
 				<topicName>/scan</topicName>
-				<frameName>laser_frame</frameName>
+				<frameName>lidar</frameName>
 			</plugin>
 		</sensor>
 	</gazebo>
-	<joint name="head_to_laser_frame" type="fixed">
-    <parent link="head"/>
-    <child link="laser_frame"/>
-    <origin xyz="${.707*width+0.04} 0 ${.707*width}"/>
+	<joint name="base_to_lidar" type="fixed">
+    <parent link="base_link"/>
+    <child link="lidar"/>
+    <origin xyz="0 0 ${(robot_side/2+lidar_height)/2}"/>
   </joint>
-  <!-- Gazebo plugin for ROS Control -->
   <gazebo>
     <plugin name="gazebo_ros_control" filename="libgazebo_ros_control.so">

Commit message: one back wheel on robot urdf

File: src/rviz_demo/urdf/robot.urdf.xacro (robot description, xacro)
@@ -4,5 +4,5 @@
   <xacro:property name="lidar_radius" value="0.06" />
   <xacro:property name="lidar_height" value="0.12" />
-  <xacro:property name="wheeldiam" value="0.07" />
+  <xacro:property name="wheeldiam" value="0.14" />
   <xacro:property name="pi" value="3.1415" />
   <material name="blue">
@@ -24,5 +24,5 @@
     <visual>
       <geometry>
-        <box size="${robot_side} ${robot_side} ${robot_side/2}"/>
+        <box size="${robot_side*2} ${robot_side} ${robot_side/2}"/>
       </geometry>
       <material name="blue"/>
@@ -30,11 +30,37 @@
     <collision>
       <geometry>
-        <box size="${robot_side} ${robot_side} ${robot_side/2}"/>
+        <box size="${robot_side*2} ${robot_side} ${robot_side/2}"/>
       </geometry>
     </collision>
     <xacro:default_inertial mass="30"/>
   </link>
-  <xacro:macro name="wheel" params="rl fb rl_reflect fb_reflect">
-    <link name="${rl}_${fb}_wheel">
+	<link name="back_wheel">
+		<visual>
+			<geometry>
+				<sphere radius="${wheeldiam/2}"/>
+			</geometry>
+		</visual>
+		<collision>
+			<geometry>
+				<sphere radius="${wheeldiam/2}"/>
+			</geometry>
+		</collision>
+		<xacro:default_inertial mass="1"/>
+	</link>
+	<joint name="base_to_back_wheel" type="continuous">
+  	<axis xyz="0 1 0" rpy="0 0 0" />
+    <parent link="base_link"/>
+    <child link="back_wheel"/>
+    <origin xyz="-${2*robot_side/3} 0 -${robot_side/4}" rpy="0 0 0"/>
+  </joint>
+  <gazebo reference="back_wheel">
+    <mu1 value="200.0"/>
+    <mu2 value="100.0"/>
+    <kp value="10000000.0" />
+    <kd value="1.0" />
+    <material>Gazebo/Grey</material>
+  </gazebo>
+  <xacro:macro name="wheel" params="rl rl_reflect">
+    <link name="${rl}_wheel">
       <visual>
         <origin xyz="0 0 0" rpy="${pi/2} 0 0" />
@@ -52,11 +78,11 @@
       <xacro:default_inertial mass="1"/>
     </link>
-    <joint name="${rl}_${fb}_wheel_joint" type="continuous">
+    <joint name="${rl}_wheel_joint" type="continuous">
       <axis xyz="0 1 0" rpy="0 0 0" />
       <parent link="base_link"/>
-      <child link="${rl}_${fb}_wheel"/>
-      <origin xyz="${robot_side/3*fb_reflect} ${robot_side/3*rl_reflect} -${wheeldiam/2+.05}" rpy="0 0 0"/>
+      <child link="${rl}_wheel"/>
+      <origin xyz="${robot_side/2} ${rl_reflect*robot_side/2} -${robot_side/4}" rpy="0 0 0"/>
     </joint>
-    <gazebo reference="${rl}_${fb}_wheel">
+    <gazebo reference="${rl}_wheel">
       <mu1 value="200.0"/>
       <mu2 value="100.0"/>
@@ -65,18 +91,16 @@
       <material>Gazebo/Grey</material>
     </gazebo>
-    <transmission name="${rl}_${fb}_wheel_trans">
+    <transmission name="${rl}_wheel_trans">
       <type>transmission_interface/SimpleTransmission</type>
-      <actuator name="${rl}_${fb}_wheel_motor">
+      <actuator name="${rl}_wheel_motor">
         <mechanicalReduction>1</mechanicalReduction>
       </actuator>
-      <joint name="${rl}_${fb}_wheel_joint">
+      <joint name="${rl}_wheel_joint">
         <hardwareInterface>VelocityJointInterface</hardwareInterface>
       </joint>
     </transmission>
   </xacro:macro>
-	<xacro:wheel rl="right" fb="front" rl_reflect="1" fb_reflect="1"/>
-	<xacro:wheel rl="right" fb="back" rl_reflect="1" fb_reflect="-1"/>
-	<xacro:wheel rl="left" fb="front" rl_reflect="-1" fb_reflect="1"/>
-	<xacro:wheel rl="left" fb="back" rl_reflect="-1" fb_reflect="-1"/>
+	<xacro:wheel rl="right"  rl_reflect="1"/>
+	<xacro:wheel rl="left" rl_reflect="-1"/>
   <link name="lidar">
     <visual>
