Commit message: turtlebot3_world working with gmapping and localization

File: src/rviz_demo/urdf/lidar.xacro (robot description, xacro)
@@ -1,23 +1,55 @@
 <?xml version="1.0"?>
-<robot xmlns:xacro="http://www.ros.org/wiki/xacro" >
-	<joint name="laser_joint" type="fixed">
-		<parent link="chassis"/>
-		<child link="laser_frame"/>
-		<origin xyz="0.1 0 0.175" rpy="0 0 0"/>
-	</joint>
-	<link name="laser_frame">
+<robot name="lidar" xmlns:xacro="http://www.ros.org/wiki/xacro" >
+<xacro:property name="lidar_radius" value="0.06" />
+<xacro:property name="lidar_height" value="0.12" />
+<xacro:macro name="lidar" params="location parent">
+	<link name="lidar">
 		<visual>
 			<geometry>
-				<cylinder radius="0.05" length="0.04"/>
+				<cylinder radius="${lidar_radius}" length="${lidar_height}" />
 			</geometry>
+			<origin xyz="0 0 0"/>
 		</visual>
 		<collision>
 			<geometry>
-				<cylinder radius="0.05" length="0.04"/>
+				<cylinder radius="${lidar_radius}" length="${lidar_height}" />
 			</geometry>
 		</collision>
-		<xacro:inertial_cylinder mass="0.1" length="0.04" radius="0.05">
-			<origin xyz="0 0 0" rpy="0 0 0"/>
-		</xacro:inertial_cylinder>
+		<inertial>
+			<mass value="1" />
+			<inertia ixx="0.1" ixy="0" ixz="0" iyy="0.1" iyz="0" izz="0.1" />
+		</inertial>
 	</link>
+	<gazebo reference="lidar">
+		<sensor name="laser" type="ray">
+			<pose>0 0 0 0 0 0</pose>
+			<visualize>true</visualize>
+			<update_rate>10</update_rate>
+			<ray>
+				<scan>
+					<horizontal>
+						<samples>360</samples>
+						<resolution>1</resolution>
+						<min_angle>-3.14</min_angle>
+						<max_angle>3.14</max_angle>
+					</horizontal>
+				</scan>
+				<range>
+					<min>0.3</min>
+					<max>12</max>
+					<resolution>0.01</resolution>
+				</range>
+			</ray>
+			<plugin name="laser_controller" filename="libgazebo_ros_laser.so">
+				<topicName>/scan</topicName>
+				<frameName>lidar</frameName>
+			</plugin>
+		</sensor>
+	</gazebo>
+	<joint name="base_to_lidar" type="fixed">
+		<parent link="base_link"/>
+		<child link="lidar"/>
+		<origin xyz="0 0 ${(robot_side/2+lidar_height)/2}"/>
+  	</joint>
+</xacro:macro>
 </robot>
